Commit message: finalised the gazebo launch file

File: src/bumperbot_description/urdf/bumperbot.urdf.xacro (robot description, xacro)
@@ -1,5 +1,10 @@
 <?xml version="1.0"?>
 <robot name="bumperbot" xmlns:xacro="http://ros.org/wiki/xacro">
+  <!-- Start GZ or Ignition depending on ROS 2 Version -->
+  <xacro:arg name="is_ignition" default="true"/>
+  <!-- Include Gazebo Parameters -->
   <xacro:include filename="$(find bumperbot_description)/urdf/bumperbot_gazebo.xacro" />
+  <!-- Include ros2_control Plugins -->
+  <xacro:include filename="$(find bumperbot_description)/urdf/bumperbot_ros2_control.xacro" />
   <link name="base_footprint"/>
   <link name="base_link">
@@ -138,18 +143,3 @@
     <axis xyz="0 0 0" />
   </joint>
-  <!-- This was an assignment to add a link of can -->
-    <!-- <link name = "can_link" type="fixed">
-        <visual>
-            <origin xyz="-0.032 .032 .079" rpy="1.57 0.0 0.0"/>
-            <geometry>
-                <mesh filename="package://bumperbot_description/meshes/can.STL" scale="1.0 1.0 1.0"/>
-            </geometry>
-        </visual>
-    </link>
-    <joint name="can_to_base" type="fixed">
-        <parent link="base_link"/>
-        <child link="can_link"/>
-        <origin xyz="0.0 0.0 0" rpy="0.0 0.0 0.0"/>
-        <axis xyz="0.0 0.0 0.0"/>
-    </joint> -->
 </robot>

File: src/bumperbot_description/urdf/bumperbot_gazebo.xacro (robot description, xacro)
@@ -35,3 +35,18 @@
         <maxVel>.1</maxVel>
     </gazebo>
+    <!-- ROS 2 Control -->
+  <gazebo>
+    <!-- ROS 2 Humble -->
+    <xacro:if value="$(arg is_ignition)">
+      <plugin filename="ign_ros2_control-system" name="ign_ros2_control::IgnitionROS2ControlPlugin">
+        <parameters>$(find bumperbot_controller)/config/bumperbot_controllers.yaml</parameters>
+      </plugin>
+    </xacro:if>
+    <!-- ROS 2 Iron or above -->
+    <xacro:unless value="$(arg is_ignition)">
+      <plugin filename="gz_ros2_control-system" name="gz_ros2_control::GazeboSimROS2ControlPlugin">
+        <parameters>$(find bumperbot_controller)/config/bumperbot_controllers.yaml</parameters>
+      </plugin>
+    </xacro:unless>
+  </gazebo>
 </robot>
