Commit message: Added the Laser_sensor to the robot

File: install/bumperbot_description/share/bumperbot_description/urdf/bumperbot.urdf.xacro (robot description, xacro)
@@ -165,4 +165,28 @@
     </collision>
   </link>
+  <!-- <link name="lidar_link">
+  <inertial>
+    <origin xyz="0 0 0.1" rpy="0 0 0" />
+    <mass value="0.2" />
+    <inertia ixx="0.0002083" ixy="0.0" ixz="0.0"
+             iyy="0.0002083" iyz="0.0"
+             izz="0.0003333" />
+  </inertial>
+  <visual>
+    <origin xyz="0 0 0" rpy="0 0 0" />
+    <geometry>
+      <mesh filename="package://bumperbot_description/meshes/LD19.STL" />
+    </geometry>
+    <material name="">
+      <color rgba="0.792156862745098 0.819607843137255 0.933333333333333 1" />
+    </material>
+  </visual>
+  <collision>
+    <origin xyz="0 0 0" rpy="0 0 0" />
+    <geometry>
+      <mesh filename="package://bumperbot_description/meshes/LD19.STL" />
+    </geometry>
+  </collision>
+</link> -->
   <joint name="imu_joint" type="fixed">
     <origin xyz="0 0 0.0698986241758014" rpy="0 0 0" />
@@ -171,3 +195,34 @@
     <axis xyz="0 0 0" />
   </joint>
+ <!-- LiDAR Link Definition with Scaled Mesh -->
+<link name="laser_link">
+  <inertial>
+    <origin xyz="-0.011945780406062 -0.000381929217680526 -0.0170649378129477" rpy="0 0 0" />
+    <mass value="0.073084435549317" />
+    <inertia ixx="1.96074931730795E-05" ixy="-3.62091076640009E-07" ixz="4.28230084046735E-07" iyy="2.40983835136327E-05" iyz="1.50180909250652E-08" izz="4.14184164228595E-05" />
+</inertial>
+  <visual>
+    <origin xyz="0 0 0" rpy="0 0 0" />
+    <geometry>
+      <!-- Scaling the mesh to 1/100 of its original dimensions -->
+      <mesh filename="package://bumperbot_description/meshes/laser_link.STL" scale="1 1 1" />
+    </geometry>
+    <material name="">
+      <color rgba="0.792156862745098 0.819607843137255 0.933333333333333 1" />
+    </material>
+  </visual>
+  <collision>
+    <origin xyz="0 0 0" rpy="0 0 0" />
+    <geometry>
+      <!-- Scaling the mesh to 1/100 of its original dimensions -->
+      <mesh filename="package://bumperbot_description/meshes/laser_link.STL" scale="1 1 1" />
+    </geometry>
+  </collision>
+</link>
+<!-- Fixed Joint to Attach the LiDAR to the Base Link -->
+  <joint name="laser_joint" type="fixed">
+    <origin xyz="0 0 0.12" rpy="0 0 3.14" />
+    <parent link="base_link" />
+    <child link="laser_link" />
+  </joint>
 </robot>

File: install/bumperbot_description/share/bumperbot_description/urdf/bumperbot_gazebo.xacro (robot description, xacro)
@@ -1,39 +1,39 @@
 <?xml version="1.0"?>
-<robot name="bumperbot" xmlns:xacro = "http://www.ros.org/wiki/xacro" >
-    <gazebo reference="wheel_right_link">
-        <mu1>100000000000000.0</mu1>
-        <mu2>100000000000000.0</mu2>
-        <kp>10000000000.0</kp>
-        <kd>10.0</kd>
-        <minDepth>.001</minDepth>
-        <maxVel>.1</maxVel>
-        <fdir1>1 0 0</fdir1>
-    </gazebo>
-    <gazebo reference="wheel_left_link">
-        <mu1>100000000000000.0</mu1>
-        <mu2>100000000000000.0</mu2>
-        <kp>10000000000.0</kp>
-        <kd>10.0</kd>
-        <minDepth>.001</minDepth>
-        <maxVel>.1</maxVel>
-        <fdir1>1 0 0</fdir1><!-- for setting the direction of rotation-->
-    </gazebo>
-    <gazebo reference="castor_front_link">
-        <mu1>0.1</mu1>
-        <mu2>0.1</mu2>
-        <kp>1000000.0</kp>
-        <kd>100.0</kd>
-        <minDepth>.001</minDepth>
-        <maxVel>.1</maxVel>
-    </gazebo>
-    <gazebo reference="castor_rear_link">
-        <mu1>0.1</mu1>
-        <mu2>0.1</mu2>
-        <kp>1000000.0</kp>
-        <kd>100.0</kd>
-        <minDepth>.001</minDepth>
-        <maxVel>.1</maxVel>
-    </gazebo>
-    <!-- ROS 2 Control -->
+<robot name="bumperbot" xmlns:xacro="http://www.ros.org/wiki/xacro">
+  <gazebo reference="wheel_right_link">
+    <mu1>100000000000000.0</mu1>
+    <mu2>100000000000000.0</mu2>
+    <kp>10000000000.0</kp>
+    <kd>10.0</kd>
+    <minDepth>.001</minDepth>
+    <maxVel>.1</maxVel>
+    <fdir1>1 0 0</fdir1>
+  </gazebo>
+  <gazebo reference="wheel_left_link">
+    <mu1>100000000000000.0</mu1>
+    <mu2>100000000000000.0</mu2>
+    <kp>10000000000.0</kp>
+    <kd>10.0</kd>
+    <minDepth>.001</minDepth>
+    <maxVel>.1</maxVel>
+    <fdir1>1 0 0</fdir1><!-- for setting the direction of rotation-->
+  </gazebo>
+  <gazebo reference="castor_front_link">
+    <mu1>0.1</mu1>
+    <mu2>0.1</mu2>
+    <kp>1000000.0</kp>
+    <kd>100.0</kd>
+    <minDepth>.001</minDepth>
+    <maxVel>.1</maxVel>
+  </gazebo>
+  <gazebo reference="castor_rear_link">
+    <mu1>0.1</mu1>
+    <mu2>0.1</mu2>
+    <kp>1000000.0</kp>
+    <kd>100.0</kd>
+    <minDepth>.001</minDepth>
+    <maxVel>.1</maxVel>
+  </gazebo>
+  <!-- ROS 2 Control -->
   <gazebo>
     <!-- ROS 2 Humble -->
@@ -43,4 +43,7 @@
       </plugin>
       <plugin filename="ignition-gazebo-imu-system" name="ignition::gazebo::systems::Imu"/>
+      <plugin filename="ignition-gazebo-sensors-system" name="ignition::gazebo::systems::Sensors">
+        <render_engine>ogre2</render_engine>
+      </plugin>
     </xacro:if>
     <!-- ROS 2 Iron or above -->
@@ -60,5 +63,5 @@
         <angular_velocity>
           <x>
-            <noise type= "gaussian">
+            <noise type="gaussian">
               <mean>0.0</mean>
               <stddev>2e-4</stddev>
@@ -66,5 +69,5 @@
           </x>
           <y>
-            <noise type= "gaussian">
+            <noise type="gaussian">
               <mean>0.0</mean>
               <stddev>2e-4</stddev>
@@ -72,5 +75,5 @@
           </y>
           <z>
-            <noise type= "gaussian">
+            <noise type="gaussian">
               <mean>0.0</mean>
               <stddev>2e-4</stddev>
@@ -80,5 +83,5 @@
         <linear_acceleration>
           <x>
-            <noise type= "gaussian">
+            <noise type="gaussian">
               <mean>0.0</mean>
               <stddev>1.7e-2</stddev>
@@ -86,5 +89,5 @@
           </x>
           <y>
-            <noise type= "gaussian">
+            <noise type="gaussian">
               <mean>0.0</mean>
               <stddev>1.7e-2</stddev>
@@ -92,5 +95,5 @@
           </y>
           <z>
-            <noise type= "gaussian">
+            <noise type="gaussian">
               <mean>0.0</mean>
               <stddev>1.7e-2</stddev>
@@ -99,5 +102,37 @@
         </linear_acceleration>
       </imu>
-    <!-- Sensor imu -->
+      <!-- Sensor imu -->
+    </sensor>
+  </gazebo>
+  <gazebo reference = "laser_link">
+    <sensor name="lidar" type="gpu_ray" >
+      <parent link="base_link"/>
+      <origin xyz="0.0 0.0 0.0" rpy="0.0 0.0 0.0"/>
+      <always_on>true</always_on>
+      <visualize>true</visualize>
+      <topic>scan</topic>
+      <update_rate>10</update_rate>
+      <gz_frame_id>laser_link</gz_frame_id>
+      <!-- Sensor gpu_ray -->
+      <ray>
+        <scan>
+          <horizontal>
+            <samples>500</samples>
+            <resolution>.72</resolution>
+            <min_angle>0</min_angle>
+            <max_angle>6.28</max_angle>
+          </horizontal>
+        </scan>
+        <range>
+          <min>0.03</min>
+          <max>10</max>
+          <resolution>.02</resolution>
+        </range>
+        <noise>
+          <type>gaussian</type>
+          <mean>0.0</mean>
+          <stddev>0.01</stddev>
+        </noise>
+      </ray>
     </sensor>
   </gazebo>
